File: Lamp_Switch.sch (KiCad schematic (older format))
At the start: 11 parts

Commit message: assign footprint
Parts:
- JP?: footprint (none) -> Pin_Headers:Pin_Header_Straight_1x02_Pitch2.00mm
Changed lines of the file:
@@
 F 0 "JP?" H 4200 3200 50  0000 C CNN
 F 1 "Jumper" H 4200 2970 50  0000 C CNN
-F 2 "" H 4200 3050 50  0001 C CNN
+F 2 "Pin_Headers:Pin_Header_Straight_1x02_Pitch2.00mm" H 4200 3050 50  0001 C CNN
 F 3 "" H 4200 3050 50  0001 C CNN
 	1    4200 3050
@@
 	3750 2750 5100 2750
 Wire Wire Line
-	3750 2750 3750 3200
+	3750 2750 3750 3050
+Wire Wire Line
+	3750 3050 3750 3200
 Wire Wire Line
 	3900 3050 3750 3050
 Wire Wire Line
-	5100 3050 4500 3050
+	5100 3050 4750 3050
+Wire Wire Line
+	4750 3050 4500 3050
 Wire Wire Line
 	5100 2900 5100 3050
@@
 	6600 3500 6600 3350
 Wire Wire Line
-	6200 3500 6950 3500
+	6200 3500 6600 3500
+Wire Wire Line
+	6600 3500 6950 3500
 Wire Wire Line
 	6200 3200 6200 3500
@@
 	6600 2600 6600 2700
 Wire Wire Line
-	6200 2600 6950 2600
+	6200 2600 6600 2600
 Wire Wire Line
-	3150 2600 5100 2600
+	6600 2600 6950 2600
+Wire Wire Line
+	3150 2600 3350 2600
+Wire Wire Line
+	3350 2600 5100 2600
 Wire Wire Line
 	3350 3850 3350 2600
@@
 	4000 4800 3200 4800
 Wire Wire Line
-	4750 3050 4750 4600
+	4750 3050 4750 4350
+Wire Wire Line
+	4750 4350 4750 4600
 Wire Wire Line
 	4750 4350 5100 4350
@@
 $EndComp
 Wire Wire Line
-	6200 3850 6950 3850
+	6200 3850 6600 3850
+Wire Wire Line
+	6600 3850 6950 3850
 Wire Wire Line
 	6600 3850 6600 3950
@@
 	6200 4450 6200 4750
 Wire Wire Line
-	6200 4750 6950 4750
+	6200 4750 6600 4750
+Wire Wire Line
+	6600 4750 6950 4750
 Wire Wire Line
 	6600 4750 6600 4600
