File: Power_12V.sch (KiCad schematic (older format))
At the start: 5 parts

Commit message: assign footprint
Parts:
- D?: footprint (none) -> LEDs:LED_0603
- JP?: footprint (none) -> Pin_Headers:Pin_Header_Straight_1x02_Pitch2.00mm
- P?: footprint (none) -> auv:XT60
- R?: footprint (none) -> Resistors_SMD:R_0603
- U?: footprint (none) -> auv:UWE-xxxx
Changed lines of the file:
@@
 F 0 "U?" H 5300 3800 60  0000 C CNN
 F 1 "UWE-12/6-Q12P" H 5600 3000 60  0000 C CNN
-F 2 "" H 5650 3100 60  0000 C CNN
+F 2 "auv:UWE-xxxx" H 5550 2900 60  0000 C CNN
 F 3 "" H 5650 3100 60  0000 C CNN
 	1    5600 3400
@@
 F 0 "JP?" H 4600 3700 50  0000 C CNN
 F 1 "Jumper" H 4600 3470 50  0000 C CNN
-F 2 "" H 4600 3550 50  0001 C CNN
+F 2 "Pin_Headers:Pin_Header_Straight_1x02_Pitch2.00mm" H 4600 3550 50  0001 C CNN
 F 3 "" H 4600 3550 50  0001 C CNN
 	1    4600 3550
@@
 F 0 "D?" H 6650 3875 50  0000 L CNN
 F 1 "LED_Small" H 6525 3650 50  0000 L CNN
-F 2 "" V 6700 3750 50  0001 C CNN
+F 2 "LEDs:LED_0603" V 6700 3750 50  0001 C CNN
 F 3 "" V 6700 3750 50  0001 C CNN
 	1    6700 3750
@@
 F 0 "R?" V 6780 3350 50  0000 C CNN
 F 1 "R" V 6700 3350 50  0000 C CNN
-F 2 "" V 6630 3350 50  0001 C CNN
+F 2 "Resistors_SMD:R_0603" V 6630 3350 50  0001 C CNN
 F 3 "" H 6700 3350 50  0001 C CNN
 	1    6700 3350
@@
 F 0 "P?" H 7350 3700 50  0000 C CNN
 F 1 "XT60" H 7350 3400 50  0000 C CNN
-F 2 "" H 7350 3550 60  0000 C CNN
+F 2 "auv:XT60" H 7450 3300 60  0000 C CNN
 F 3 "" H 7350 3550 60  0000 C CNN
 	1    7350 3550
