File: Thruster_Switch.sch (KiCad schematic (older format))
At the start: 15 parts

Commit message: remove R on BJT emitter and insert 10V zener diode instead
Parts:
- removed R?: 10K, Resistors_SMD:R_0603, symbol R
- added D?: BZX384-C12, Diodes_SMD:D_SOD-323, symbol D_Zener
- added R?: 330, Resistors_SMD:R_0603, symbol R
- Q?: value IPI120P04P4L -> IPD90P03P4L; footprint TO_SOT_Packages_SMD:TO-263-3Lead -> TO_SOT_Packages_SMD:TO-252-2Lead
- R?: value 100 -> 1k
Connections:
- wire segments 30 -> 32
Other:
- moved on the sheet: C?
Changed lines of the file:
@@
 LIBS:zeabus
 LIBS:ftdi
-LIBS:Power_Distributor-cache
 EELAYER 25 0
 EELAYER END
 $Descr A4 11693 8268
 encoding utf-8
-Sheet 6 12
+Sheet 11 12
 Title ""
 Date ""
@@
 AR Path="/58E62AD5/58E01FFB" Ref="R?"  Part="1"
 F 0 "R?" V 5630 3050 50  0000 C CNN
-F 1 "100" V 5550 3050 50  0000 C CNN
+F 1 "1k" V 5550 3050 50  0000 C CNN
 F 2 "Resistors_SMD:R_0603" V 5480 3050 50  0001 C CNN
 F 3 "" H 5550 3050 50  0001 C CNN
@@
 L C C?
 U 1 1 58E53CD9
-P 4600 4350
+P 4500 4350
 AR Path="/58E0048C/58E53CD9" Ref="C?"  Part="1"
 AR Path="/58E52973/58E53CD9" Ref="C?"  Part="1"
 AR Path="/58E62AD5/58E53CD9" Ref="C?"  Part="1"
-F 0 "C?" H 4625 4450 50  0000 L CNN
-F 1 "1uF" H 4625 4250 50  0000 L CNN
-F 2 "Capacitors_SMD:C_0603" H 4638 4200 50  0001 C CNN
-F 3 "" H 4600 4350 50  0001 C CNN
-	1    4600 4350
+F 0 "C?" H 4525 4450 50  0000 L CNN
+F 1 "1uF" H 4525 4250 50  0000 L CNN
+F 2 "Capacitors_SMD:C_0603" H 4538 4200 50  0001 C CNN
+F 3 "" H 4500 4350 50  0001 C CNN
+	1    4500 4350
 	1    0    0    -1
 $EndComp
@@
 Wire Wire Line
 	4250 4650 4250 4500
-Wire Wire Line
-	4600 4050 4600 4200
-Connection ~ 4600 4050
-Wire Wire Line
-	4600 4500 4600 4750
 $Comp
 L Q_PMOS_GDS Q?
@@
 AR Path="/58E62AD5/58E51C6A" Ref="Q?"  Part="1"
 F 0 "Q?" H 6350 3100 50  0000 L CNN
-F 1 "IPI120P04P4L" H 6350 3000 50  0000 L CNN
-F 2 "TO_SOT_Packages_SMD:TO-263-3Lead" H 6350 3150 50  0001 C CNN
+F 1 "IPD90P03P4L" H 6350 3000 50  0000 L CNN
+F 2 "TO_SOT_Packages_SMD:TO-252-2Lead" H 6350 3150 50  0001 C CNN
 F 3 "" H 6150 3050 50  0001 C CNN
 	1    6150 3050
 	1    0    0    1
 $EndComp
-$Comp
-L R R?
-U 1 1 58E67103
-P 5250 4500
-AR Path="/58E0048C/58E67103" Ref="R?"  Part="1"
-AR Path="/58E52973/58E67103" Ref="R?"  Part="1"
-AR Path="/58E62AD5/58E67103" Ref="R?"  Part="1"
-F 0 "R?" V 5330 4500 50  0000 C CNN
-F 1 "10K" V 5250 4500 50  0000 C CNN
-F 2 "Resistors_SMD:R_0603" V 5180 4500 50  0001 C CNN
-F 3 "" H 5250 4500 50  0001 C CNN
-	1    5250 4500
-	-1   0    0    1
-$EndComp
-Wire Wire Line
-	5250 4250 5250 4350
-Wire Wire Line
-	5250 4650 5250 4900
+Wire Wire Line
+	5250 4250 5250 4900
 Wire Wire Line
 	3650 2300 6250 2300
 Wire Wire Line
-	4150 4050 4950 4050
-Wire Wire Line
-	4600 4750 8300 4750
+	4500 4750 8300 4750
+$Comp
+L R R?
+U 1 1 58E6316B
+P 4700 4050
+F 0 "R?" V 4780 4050 50  0000 C CNN
+F 1 "330" V 4700 4050 50  0000 C CNN
+F 2 "Resistors_SMD:R_0603" V 4630 4050 50  0001 C CNN
+F 3 "" H 4700 4050 50  0001 C CNN
+	1    4700 4050
+	0    -1   -1   0
+$EndComp
+Wire Wire Line
+	4500 4200 4500 4050
+Wire Wire Line
+	4150 4050 4550 4050
+Wire Wire Line
+	4850 4050 4950 4050
+Wire Wire Line
+	4500 4500 4500 4750
+Connection ~ 4500 4050
+$Comp
+L D_Zener D?
+U 1 1 58E6427A
+P 5850 2750
+F 0 "D?" H 5850 2850 50  0000 C CNN
+F 1 "BZX384-C12" H 5850 2650 50  0000 C CNN
+F 2 "Diodes_SMD:D_SOD-323" H 5850 2750 50  0001 C CNN
+F 3 "" H 5850 2750 50  0001 C CNN
+	1    5850 2750
+	0    1    1    0
+$EndComp
+Wire Wire Line
+	5850 2600 5850 2500
+Connection ~ 5850 2500
+Wire Wire Line
+	5850 2900 5850 3050
+Connection ~ 5850 3050
 $EndSCHEMATC

Commit message: change BZX-384 to BZX-585
Parts:
- D?: value BZX384-C12 -> BZX585-C12; footprint Diodes_SMD:D_SOD-323 -> Diodes_SMD:D_SOD-523
Changed lines of the file:
@@
 AR Path="/58E52973/58E019DD" Ref="P?"  Part="1"
 AR Path="/58E62AD5/58E019DD" Ref="P?"  Part="1"
+AR Path="/58E6D43E/58E019DD" Ref="P?"  Part="1"
 F 0 "P?" H 6850 4450 50  0000 C CNN
 F 1 "XT60" H 6850 4150 50  0000 C CNN
@@
 AR Path="/58E52973/58E01A68" Ref="R?"  Part="1"
 AR Path="/58E62AD5/58E01A68" Ref="R?"  Part="1"
+AR Path="/58E6D43E/58E01A68" Ref="R?"  Part="1"
 F 0 "R?" V 6330 4150 50  0000 C CNN
 F 1 "10k" V 6250 4150 50  0000 C CNN
@@
 AR Path="/58E52973/58E01A8B" Ref="D?"  Part="1"
 AR Path="/58E62AD5/58E01A8B" Ref="D?"  Part="1"
+AR Path="/58E6D43E/58E01A8B" Ref="D?"  Part="1"
 F 0 "D?" H 6200 4675 50  0000 L CNN
 F 1 "LED_Small" H 6075 4450 50  0000 L CNN
@@
 AR Path="/58E52973/58E01FA8" Ref="R?"  Part="1"
 AR Path="/58E62AD5/58E01FA8" Ref="R?"  Part="1"
+AR Path="/58E6D43E/58E01FA8" Ref="R?"  Part="1"
 F 0 "R?" V 5630 2500 50  0000 C CNN
 F 1 "10k" V 5550 2500 50  0000 C CNN
@@
 AR Path="/58E52973/58E01FFB" Ref="R?"  Part="1"
 AR Path="/58E62AD5/58E01FFB" Ref="R?"  Part="1"
+AR Path="/58E6D43E/58E01FFB" Ref="R?"  Part="1"
 F 0 "R?" V 5630 3050 50  0000 C CNN
 F 1 "1k" V 5550 3050 50  0000 C CNN
@@
 AR Path="/58E52973/58E0369B" Ref="#PWR?"  Part="1"
 AR Path="/58E62AD5/58E0369B" Ref="#PWR?"  Part="1"
+AR Path="/58E6D43E/58E0369B" Ref="#PWR?"  Part="1"
 F 0 "#PWR?" H 5250 4650 50  0001 C CNN
 F 1 "GND" H 5250 4750 50  0000 C CNN
@@
 AR Path="/58E52973/58E0D2A0" Ref="P?"  Part="1"
 AR Path="/58E62AD5/58E0D2A0" Ref="P?"  Part="1"
+AR Path="/58E6D43E/58E0D2A0" Ref="P?"  Part="1"
 F 0 "P?" H 7400 4450 50  0000 C CNN
 F 1 "XT60" H 7400 4150 50  0000 C CNN
@@
 AR Path="/58E52973/58E0D2E8" Ref="P?"  Part="1"
 AR Path="/58E62AD5/58E0D2E8" Ref="P?"  Part="1"
+AR Path="/58E6D43E/58E0D2E8" Ref="P?"  Part="1"
 F 0 "P?" H 7950 4450 50  0000 C CNN
 F 1 "XT60" H 7950 4150 50  0000 C CNN
@@
 AR Path="/58E52973/58E0D33F" Ref="P?"  Part="1"
 AR Path="/58E62AD5/58E0D33F" Ref="P?"  Part="1"
+AR Path="/58E6D43E/58E0D33F" Ref="P?"  Part="1"
 F 0 "P?" H 8500 4450 50  0000 C CNN
 F 1 "XT60" H 8500 4150 50  0000 C CNN
@@
 AR Path="/58E52973/58E4CD5F" Ref="R?"  Part="1"
 AR Path="/58E62AD5/58E4CD5F" Ref="R?"  Part="1"
+AR Path="/58E6D43E/58E4CD5F" Ref="R?"  Part="1"
 F 0 "R?" V 4080 4050 50  0000 C CNN
 F 1 "2.2k" V 4000 4050 50  0000 C CNN
@@
 AR Path="/58E52973/58E4F6EC" Ref="Q?"  Part="1"
 AR Path="/58E62AD5/58E4F6EC" Ref="Q?"  Part="1"
+AR Path="/58E6D43E/58E4F6EC" Ref="Q?"  Part="1"
 F 0 "Q?" H 5350 4125 50  0000 L CNN
 F 1 "BC817-40" H 5350 4050 50  0000 L CNN
@@
 AR Path="/58E52973/58E4FE30" Ref="F?"  Part="1"
 AR Path="/58E62AD5/58E4FE30" Ref="F?"  Part="1"
+AR Path="/58E6D43E/58E4FE30" Ref="F?"  Part="1"
 F 0 "F?" V 6330 3550 50  0000 C CNN
 F 1 "Fuse" V 6175 3550 50  0000 C CNN
@@
 AR Path="/58E52973/58E515C3" Ref="D?"  Part="1"
 AR Path="/58E62AD5/58E515C3" Ref="D?"  Part="1"
+AR Path="/58E6D43E/58E515C3" Ref="D?"  Part="1"
 F 0 "D?" H 4250 4450 50  0000 C CNN
 F 1 "MBR0530T3G" H 4250 4250 50  0000 C CNN
@@
 AR Path="/58E52973/58E53CD9" Ref="C?"  Part="1"
 AR Path="/58E62AD5/58E53CD9" Ref="C?"  Part="1"
+AR Path="/58E6D43E/58E53CD9" Ref="C?"  Part="1"
 F 0 "C?" H 4525 4450 50  0000 L CNN
 F 1 "1uF" H 4525 4250 50  0000 L CNN
@@
 AR Path="/58E52973/58E51C6A" Ref="Q?"  Part="1"
 AR Path="/58E62AD5/58E51C6A" Ref="Q?"  Part="1"
+AR Path="/58E6D43E/58E51C6A" Ref="Q?"  Part="1"
 F 0 "Q?" H 6350 3100 50  0000 L CNN
 F 1 "IPD90P03P4L" H 6350 3000 50  0000 L CNN
@@
 U 1 1 58E6316B
 P 4700 4050
+AR Path="/58E0048C/58E6316B" Ref="R?"  Part="1"
+AR Path="/58E6D43E/58E6316B" Ref="R?"  Part="1"
 F 0 "R?" V 4780 4050 50  0000 C CNN
 F 1 "330" V 4700 4050 50  0000 C CNN
@@
 U 1 1 58E6427A
 P 5850 2750
+AR Path="/58E0048C/58E6427A" Ref="D?"  Part="1"
+AR Path="/58E6D43E/58E6427A" Ref="D?"  Part="1"
 F 0 "D?" H 5850 2850 50  0000 C CNN
-F 1 "BZX384-C12" H 5850 2650 50  0000 C CNN
-F 2 "Diodes_SMD:D_SOD-323" H 5850 2750 50  0001 C CNN
+F 1 "BZX585-C12" H 5850 2650 50  0000 C CNN
+F 2 "Diodes_SMD:D_SOD-523" H 5850 2750 50  0001 C CNN
 F 3 "" H 5850 2750 50  0001 C CNN
 	1    5850 2750
