File: Power-Volt-Converter.sch (KiCad schematic (older format))
At the start: 31 parts, among them P1 XT60, P2 XT60, P3 XT60, P4 XT60, P5 XT60, P6 XT60, P7 XT60, P8 XT60, Q1 BC817-40, U1 UWE-12/6-Q12P, U2 UWE-12/6-Q12P, U3 UWE-12/6-Q12P, U4 TEN_20-2411WIN, U5 TEN_20-2411WIN

Commit message: Bug fixed and clean-up for PCB generating
Parts:
- removed R10, R3: 10k, Resistors_SMD:R_0603, symbol R
- renumbered D1 to D17, D2 to D18, D3 to D19, D4 to D20, D5 to D21, P1 to P22, P4 to P23, P5 to P24, P2 to P25, P3 to P26, P6 to P27, P8 to P28, P7 to P29, Q1 to Q15, R1 to R44, R5 to R45, R2 to R46, R4 to R47, R6 to R48, R7 to R49, R8 to R50, R9 to R51, R11 to R52, U4 to U10, U5 to U11, U1 to U7, U2 to U8, U3 to U9
Connections:
- net labels added: Lamp_SW_C, Lamp_SW_E
- net labels removed: Lamp1_SW_C, Lamp1_SW_E, Lamp2_SW_C, Lamp2_SW_E
- wire segments 79 -> 78
Other:
- moved on the sheet: D19, P24, R45, R48, U9

Commit message: Bug fixed in DC-DC Converter and removed unused files.
Parts:
- removed R49: 1k, Resistors_SMD:R_0603, symbol R
- removed R50: 10k, Resistors_SMD:R_0603, symbol R
- added D?: BZX585-C12, Diodes_SMD:D_SOD-523, symbol D_Zener
- added R?: 10k, Resistors_SMD:R_0603, symbol R
Connections:
- net labels removed: +12V
- wire segments 78 -> 81
Other:
- moved on the sheet: D18, D19, D20, D21, P23, P24, P27, P28, P29, R45, R47, R48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
