File: Power-Controller.sch (KiCad schematic (older format))
At the start: 41 parts, among them P19 USB_B, U1 93LC56BT-I/OT, U2 FT232H, U3 ACPL-247-500E, U4 ACPL-247-500E, Y1 12MHz

Commit message: update footprint of 12MHz crystal
Parts:
- Y1: footprint Crystals:Crystal_FOX-FE_SMD -> Crystals:Crystal_SMD_FOX_FE-2pin_7.5x5.0mm
Changed lines of the file:
@@
 F 0 "Y1" H 4450 5750 50  0000 C CNN
 F 1 "12MHz" H 4450 5550 50  0000 C CNN
-F 2 "Crystals:Crystal_FOX-FE_SMD" H 4450 5650 60  0001 C CNN
+F 2 "Crystals:Crystal_SMD_FOX_FE-2pin_7.5x5.0mm" H 4450 5650 60  0001 C CNN
 F 3 "" H 4450 5650 60  0000 C CNN
 	1    4450 5650

Commit message: fix wrong footprint assign on C9
Parts:
- C9: footprint MMZ1608S601A-CT -> Capacitors_SMD:C_0805
Changed lines of the file:
@@
 F 0 "C9" H 3410 2870 50  0000 L CNN
 F 1 "4.7uF" H 3410 2720 50  0000 L CNN
-F 2 "MMZ1608S601A-CT" H 3400 2800 50  0001 C CNN
+F 2 "Capacitors_SMD:C_0805" H 3400 2800 50  0001 C CNN
 F 3 "" H 3400 2800 50  0000 C CNN
 	1    3400 2800

Commit message: Update Netlist
Parts:
- renumbered C7 to C1, C16 to C10, C17 to C11, C18 to C12, C19 to C13, C20 to C14, C21 to C15, C22 to C16, C23 to C17, C24 to C18, C8 to C2, C9 to C3, C10 to C4, C11 to C5, C12 to C6, C13 to C7, C14 to C8, C15 to C9, R31 to R19, R32 to R20, R33 to R21, R34 to R22, R35 to R23, R36 to R24, R37 to R25, R38 to R26, R39 to R27, R40 to R28, R41 to R29, R42 to R30, R43 to R31

Commit message: Correct GND mixed-up and re-route USB signals as a differential pairs with match length.
Connections:
- net labels added: D+, D-, GNDD
- net labels removed: GND
- no-connect marks 0 -> 11

Commit message: Bug fixed
Connections:
- wire segments 157 -> 158
Other:
- moved on the sheet: R19, R20, R21, R22
Changed lines of the file:
@@
 LIBS:zeabus
 LIBS:ftdi
-LIBS:Power_Distributor-cache
 EELAYER 25 0
 EELAYER END
@@
 L R R21
 U 1 1 58C6363A
+P 3800 4500
+F 0 "R21" V 3880 4500 50  0000 C CNN
+F 1 "10k" V 3800 4500 50  0000 C CNN
+F 2 "Resistors_SMD:R_0603" V 3730 4500 30  0001 C CNN
+F 3 "" H 3800 4500 30  0000 C CNN
+	1    3800 4500
+	-1   0    0    1
+$EndComp
+$Comp
+L R R22
+U 1 1 58C636B2
+P 3400 4500
+F 0 "R22" V 3480 4500 50  0000 C CNN
+F 1 "10k" V 3400 4500 50  0000 C CNN
+F 2 "Resistors_SMD:R_0603" V 3330 4500 30  0001 C CNN
+F 3 "" H 3400 4500 30  0000 C CNN
+	1    3400 4500
+	-1   0    0    1
+$EndComp
+$Comp
+L R R19
+U 1 1 58C63700
 P 3600 4500
-F 0 "R21" V 3680 4500 50  0000 C CNN
+F 0 "R19" V 3680 4500 50  0000 C CNN
 F 1 "10k" V 3600 4500 50  0000 C CNN
 F 2 "Resistors_SMD:R_0603" V 3530 4500 30  0001 C CNN
@@
 $EndComp
 $Comp
-L R R22
-U 1 1 58C636B2
-P 3800 4500
-F 0 "R22" V 3880 4500 50  0000 C CNN
-F 1 "10k" V 3800 4500 50  0000 C CNN
-F 2 "Resistors_SMD:R_0603" V 3730 4500 30  0001 C CNN
-F 3 "" H 3800 4500 30  0000 C CNN
-	1    3800 4500
-	-1   0    0    1
-$EndComp
-$Comp
-L R R19
-U 1 1 58C63700
-P 3400 4500
-F 0 "R19" V 3480 4500 50  0000 C CNN
-F 1 "10k" V 3400 4500 50  0000 C CNN
-F 2 "Resistors_SMD:R_0603" V 3330 4500 30  0001 C CNN
-F 3 "" H 3400 4500 30  0000 C CNN
-	1    3400 4500
-	-1   0    0    1
-$EndComp
-$Comp
 L R R20
 U 1 1 58C63845
-P 3550 5050
-F 0 "R20" V 3450 5050 50  0000 C CNN
-F 1 "2.2k" V 3550 5050 50  0000 C CNN
-F 2 "Resistors_SMD:R_0603" V 3480 5050 30  0001 C CNN
-F 3 "" H 3550 5050 30  0000 C CNN
-	1    3550 5050
+P 3600 5050
+F 0 "R20" V 3500 5050 50  0000 C CNN
+F 1 "2.2k" V 3600 5050 50  0000 C CNN
+F 2 "Resistors_SMD:R_0603" V 3530 5050 30  0001 C CNN
+F 3 "" H 3600 5050 30  0000 C CNN
+	1    3600 5050
 	0    -1   -1   0
 $EndComp
@@
 	3950 4450 5000 4450
 Wire Wire Line
-	3300 5050 3400 5050
-Wire Wire Line
-	3800 5050 3700 5050
-Wire Wire Line
-	3800 4650 3800 5050
-Connection ~ 3800 4950
-Wire Wire Line
-	3600 4650 3600 4850
-Connection ~ 3600 4850
-Wire Wire Line
-	3400 4650 3400 4750
-Connection ~ 3400 4750
+	3300 5050 3450 5050
+Wire Wire Line
+	3800 4950 3800 5050
+Connection ~ 3800 4850
+Connection ~ 3600 4750
 $Comp
 L C_Small C1
@@
 	2450 3550 2250 3550
 Wire Wire Line
-	1950 2950 1950 2900
-Wire Wire Line
-	1950 2900 1450 2900
+	1950 2900 1950 2950
+Wire Wire Line
+	1450 2900 1950 2900
 Wire Wire Line
 	1450 2900 1450 2950
@@
 Text Label 3400 3350 0    60   ~ 0
 D+
+Connection ~ 3800 4950
+Wire Wire Line
+	3600 4650 3600 4750
+Wire Wire Line
+	3800 4650 3800 4850
+Wire Wire Line
+	3400 5050 3400 4650
+Connection ~ 3400 5050
+Wire Wire Line
+	3800 5050 3750 5050
 $EndSCHEMATC
